File: ESP32S3_Board.kicad_pcb (KiCad board)
At the start: 4 copper layers, 18.4 x 23.6 mm, 31 parts, among them J1 USB_C_Receptacle_USB2.0, J2 Conn_01x08, J3 Conn_01x08, SW1 RESET, SW2 BOOT, U1 ESP32-S3FH4R2, U2 AP2112K-3.3, Y1 40MHz

Commit message: manufacturing v2
Parts:
- L1: footprint Inductor_SMD:L_0201_0603Metric -> Inductor_SMD:L_0402_1005Metric
Changed lines of the file:
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@@
     )
   )
-  (footprint "Inductor_SMD:L_0201_0603Metric" (layer "B.Cu")
+  (footprint "Inductor_SMD:L_0402_1005Metric" (layer "B.Cu")
     (at 140.528 92.202)
-    (descr "Inductor SMD 0201 (0603 Metric), square (rectangular) end terminal, IPC_7351 nominal, (Body size source: https://www.vishay.com/docs/20052/crcw0201e3.pdf), generated with kicad-footprint-generator")
+    (descr "Inductor SMD 0402 (1005 Metric), square (rectangular) end terminal, IPC_7351 nominal, (Body size source: http://www.tortai-tech.com/upload/download/2011102023233369053.pdf), generated with kicad-footprint-generator")
     (tags "inductor")
     (property "Sheetfile" "ESP32S3_Board.kicad_sch")
@@
     (property "ki_keywords" "inductor choke coil reactor magnetic")
     (attr smd)
-    (fp_text reference "L1" (at 0 1.858) (layer "B.SilkS") hide
-        (effects (font (size 1 1) (thickness 0.15)) (justify mirror))
-    )
-    (fp_text value "2nH" (at 0 -1.05) (layer "B.Fab")
-        (effects (font (size 1 1) (thickness 0.15)) (justify mirror))
-    )
-    (fp_text user "${REFERENCE}" (at 0 0.68) (layer "B.Fab")
+    (fp_text reference "L1" (at 0 1.17 180) (layer "B.SilkS")
+        (effects (font (size 1 1) (thickness 0.15)) (justify mirror))
+    )
+    (fp_text value "2nH" (at 0 -1.17 180) (layer "B.Fab")
+        (effects (font (size 1 1) (thickness 0.15)) (justify mirror))
+    )
+    (fp_text user "${REFERENCE}" (at 0 0 180) (layer "B.Fab")
         (effects (font (size 0.25 0.25) (thickness 0.04)) (justify mirror))
     )
-    (fp_line (start -0.7 -0.35) (end -0.7 0.35)
-      (stroke (width 0.05) (type solid)) (layer "B.CrtYd"))
-    (fp_line (start -0.7 0.35) (end 0.7 0.35)
-      (stroke (width 0.05) (type solid)) (layer "B.CrtYd"))
-    (fp_line (start 0.7 -0.35) (end -0.7 -0.35)
-      (stroke (width 0.05) (type solid)) (layer "B.CrtYd"))
-    (fp_line (start 0.7 0.35) (end 0.7 -0.35)
-      (stroke (width 0.05) (type solid)) (layer "B.CrtYd"))
-    (fp_line (start -0.3 -0.15) (end -0.3 0.15)
-      (stroke (width 0.1) (type solid)) (layer "B.Fab"))
-    (fp_line (start -0.3 0.15) (end 0.3 0.15)
-      (stroke (width 0.1) (type solid)) (layer "B.Fab"))
-    (fp_line (start 0.3 -0.15) (end -0.3 -0.15)
-      (stroke (width 0.1) (type solid)) (layer "B.Fab"))
-    (fp_line (start 0.3 0.15) (end 0.3 -0.15)
-      (stroke (width 0.1) (type solid)) (layer "B.Fab"))
-    (pad "" smd roundrect (at -0.345 0) (size 0.318 0.36) (layers "B.Paste") (roundrect_rratio 0.25))
-    (pad "" smd roundrect (at 0.345 0) (size 0.318 0.36) (layers "B.Paste") (roundrect_rratio 0.25))
-    (pad "1" smd roundrect (at -0.32 0) (size 0.46 0.4) (layers "B.Cu" "B.Mask") (roundrect_rratio 0.25)
+    (fp_line (start -0.93 -0.47) (end -0.93 0.47)
+      (stroke (width 0.05) (type solid)) (layer "B.CrtYd"))
+    (fp_line (start -0.93 0.47) (end 0.93 0.47)
+      (stroke (width 0.05) (type solid)) (layer "B.CrtYd"))
+    (fp_line (start 0.93 -0.47) (end -0.93 -0.47)
+      (stroke (width 0.05) (type solid)) (layer "B.CrtYd"))
+    (fp_line (start 0.93 0.47) (end 0.93 -0.47)
+      (stroke (width 0.05) (type solid)) (layer "B.CrtYd"))
+    (fp_line (start -0.5 -0.25) (end -0.5 0.25)
+      (stroke (width 0.1) (type solid)) (layer "B.Fab"))
+    (fp_line (start -0.5 0.25) (end 0.5 0.25)
+      (stroke (width 0.1) (type solid)) (layer "B.Fab"))
+    (fp_line (start 0.5 -0.25) (end -0.5 -0.25)
+      (stroke (width 0.1) (type solid)) (layer "B.Fab"))
+    (fp_line (start 0.5 0.25) (end 0.5 -0.25)
+      (stroke (width 0.1) (type solid)) (layer "B.Fab"))
+    (pad "1" smd roundrect (at -0.485 0) (size 0.59 0.64) (layers "B.Cu" "B.Paste" "B.Mask") (roundrect_rratio 0.25)
       (net 6 "+3.3V") (pinfunction "1") (pintype "passive"))
-    (pad "2" smd roundrect (at 0.32 0) (size 0.46 0.4) (layers "B.Cu" "B.Mask") (roundrect_rratio 0.25)
+    (pad "2" smd roundrect (at 0.485 0) (size 0.59 0.64) (layers "B.Cu" "B.Paste" "B.Mask") (roundrect_rratio 0.25)
       (net 2 "Net-(C4-Pad1)") (pinfunction "2") (pintype "passive"))
-    (model "${KICAD6_3DMODEL_DIR}/Inductor_SMD.3dshapes/L_0201_0603Metric.wrl"
+    (model "${KICAD6_3DMODEL_DIR}/Inductor_SMD.3dshapes/L_0402_1005Metric.wrl"
       (offset (xyz 0 0 0))
       (scale (xyz 1 1 1))
@@
   (segment (start 141.066 91.062) (end 140.942 91.186) (width 0.2) (layer "B.Cu") (net 2))
   (segment (start 142.024 91.062) (end 141.066 91.062) (width 0.2) (layer "B.Cu") (net 2))
-  (segment (start 140.540028 92.044028) (end 140.868 92.372) (width 0.2) (layer "F.Cu") (net 3))
-  (segment (start 139.428929 92.044028) (end 140.540028 92.044028) (width 0.2) (layer "F.Cu") (net 3))
   (segment (start 144.628 91.768) (end 144.3 91.44) (width 0.3) (layer "F.Cu") (net 3))
   (segment (start 139.7 92.962) (end 140.278 92.962) (width 0.3) (layer "F.Cu") (net 3))
+  (segment (start 139.077729 91.325729) (end 139.821729 91.325729) (width 0.2) (layer "F.Cu") (net 3))
+  (segment (start 139.821729 91.325729) (end 140.868 92.372) (width 0.2) (layer "F.Cu") (net 3))
   (segment (start 140.278 92.962) (end 140.868 92.372) (width 0.3) (layer "F.Cu") (net 3))
   (segment (start 144.628 92.372) (end 144.628 91.768) (width 0.3) (layer "F.Cu") (net 3))
   (segment (start 140.868 92.372) (end 144.628 92.372) (width 0.3) (layer "F.Cu") (net 3))
-  (via (at 139.428929 92.044028) (size 0.7) (drill 0.3) (layers "F.Cu" "B.Cu") (net 3))
-  (segment (start 140.612 89.812) (end 140.485 89.812) (width 0.2) (layer "B.Cu") (net 3))
-  (segment (start 139.827 89.408) (end 139.58 89.655) (width 0.2) (layer "B.Cu") (net 3))
-  (segment (start 139.58 90.470609) (end 139.192 90.858609) (width 0.2) (layer "B.Cu") (net 3))
-  (segment (start 142.024 90.662) (end 141.462 90.662) (width 0.2) (layer "B.Cu") (net 3))
-  (segment (start 140.081 89.408) (end 139.827 89.408) (width 0.2) (layer "B.Cu") (net 3))
-  (segment (start 139.192 90.858609) (end 139.192 91.807099) (width 0.2) (layer "B.Cu") (net 3))
-  (segment (start 139.58 89.655) (end 139.58 90.470609) (width 0.2) (layer "B.Cu") (net 3))
-  (segment (start 141.462 90.662) (end 140.612 89.812) (width 0.2) (layer "B.Cu") (net 3))
-  (segment (start 139.192 91.807099) (end 139.428929 92.044028) (width 0.2) (layer "B.Cu") (net 3))
-  (segment (start 140.485 89.812) (end 140.081 89.408) (width 0.2) (layer "B.Cu") (net 3))
+  (via (at 139.077729 91.325729) (size 0.7) (drill 0.3) (layers "F.Cu" "B.Cu") (net 3))
+  (segment (start 140.081 89.408) (end 140.485 89.812) (width 0.2) (layer "B.Cu") (net 3))
+  (segment (start 139.077729 91.325729) (end 139.192 91.211458) (width 0.2) (layer "B.Cu") (net 3))
+  (segment (start 140.612 89.812) (end 141.462 90.662) (width 0.2) (layer "B.Cu") (net 3))
+  (segment (start 139.192 90.858609) (end 139.58 90.470609) (width 0.2) (layer "B.Cu") (net 3))
+  (segment (start 141.462 90.662) (end 142.024 90.662) (width 0.2) (layer "B.Cu") (net 3))
+  (segment (start 139.192 91.211458) (end 139.192 90.858609) (width 0.2) (layer "B.Cu") (net 3))
+  (segment (start 139.58 89.655) (end 139.827 89.408) (width 0.2) (layer "B.Cu") (net 3))
+  (segment (start 139.827 89.408) (end 140.081 89.408) (width 0.2) (layer "B.Cu") (net 3))
+  (segment (start 139.58 90.470609) (end 139.58 89.655) (width 0.2) (layer "B.Cu") (net 3))
+  (segment (start 140.485 89.812) (end 140.612 89.812) (width 0.2) (layer "B.Cu") (net 3))
   (segment (start 147.740965 93.541035) (end 146.71 94.572) (width 0.2) (layer "F.Cu") (net 4))
   (segment (start 146.71 94.572) (end 150.47 94.572) (width 0.3) (layer "F.Cu") (net 4))
@@
   (via (at 142.876042 87.504042) (size 0.7) (drill 0.3) (layers "F.Cu" "B.Cu") (net 6))
   (via (at 151.384 93.599) (size 0.7) (drill 0.3) (layers "F.Cu" "B.Cu") (net 6))
-  (segment (start 140.208 92.71) (end 140.208 92.202) (width 0.3) (layer "B.Cu") (net 6))
   (segment (start 145.490076 97.663) (end 145.542 97.663) (width 0.3) (layer "B.Cu") (net 6))
   (segment (start 144.834 84.89) (end 144.78 84.836) (width 0.2) (layer "B.Cu") (net 6))
@@
   (segment (start 150.622 94.361) (end 147.983 94.361) (width 0.3) (layer "B.Cu") (net 6))
   (segment (start 142.834 92.672) (end 143.184 92.672) (width 0.3) (layer "B.Cu") (net 6))
+  (segment (start 139.7 93.218) (end 139.7 92.692196) (width 0.3) (layer "B.Cu") (net 6))
+  (segment (start 139.7 92.692196) (end 140.190196 92.202) (width 0.3) (layer "B.Cu") (net 6))
   (segment (start 142.876042 87.319958) (end 142.876042 87.504042) (width 0.2) (layer "B.Cu") (net 6))
   (segment (start 144.834 86.382) (end 144.475 86.741) (width 0.2) (layer "B.Cu") (net 6))
@@
   (segment (start 139.756 94.234) (end 138.846 94.234) (width 0.3) (layer "B.Cu") (net 6))
   (segment (start 143.048846 94.008) (end 144.018 94.977154) (width 0.3) (layer "B.Cu") (net 6))
-  (segment (start 139.7 93.218) (end 140.208 92.71) (width 0.3) (layer "B.Cu") (net 6))
   (segment (start 144.475 86.741) (end 143.455 86.741) (width 0.2) (layer "B.Cu") (net 6))
   (segment (start 144.834 85.852) (end 144.834 86.382) (width 0.2) (layer "B.Cu") (net 6))
