File: ESP32S3_Board.kicad_sch (KiCad schematic)
At the start: 31 parts, among them J1 USB_C_Receptacle_USB2.0, J2 Conn_01x08, J3 Conn_01x08, SW1 RESET, SW2 BOOT, U1 ESP32-S3FH4R2, U2 AP2112K-3.3, Y1 40MHz

Commit message: manufacturing v2
Parts:
- L1: footprint Inductor_SMD:L_0201_0603Metric -> Inductor_SMD:L_0402_1005Metric
Other:
- note added: "FIX THIS"
